Commit message: updating the robot model

File: dev_ws/src/field_robot/robot_description/tb3/turtlebot3_burger_for_pumpkin.urdf.xacro (robot description, xacro)
@@ -1,6 +1,4 @@
 <?xml version="1.0" ?>
 <robot name="turtlebot3_burger_for_autorace" xmlns:xacro="http://ros.org/wiki/xacro">
-  <xacro:arg name="laser_visual" default="true"/>
-  <xacro:arg name="camera_visual" default="true"/>
   <!-- Init colour -->
   <material name="black">
@@ -23,8 +21,8 @@
   </material>
   <material name="orange">
-    <color rgba="${255/255} ${108/255} ${10/255} 1.0"/>
+    <color rgba="1.0 0.42 0.04 1.0"/>
   </material>
   <material name="brown">
-    <color rgba="${222/255} ${207/255} ${195/255} 1.0"/>
+    <color rgba="1.0 0.81 0.76 1.0"/>
   </material>
   <material name="red">
@@ -89,32 +87,30 @@
   </gazebo>
   <!--link : https://www.raspberrypi.org/documentation/hardware/camera/-->
-  <gazebo reference="camera_rgb_frame">
-    <sensor type="camera" name="PiCamera">
-      <always_on>true</always_on>
-		<!-- visualize wird oben auf true/false gesetzt -->
-      <visualize>true</visualize>
-      <camera>
-		  <!-- The horizontal field of view of the camera in radians -->
-			<!-- Pi Fisheye Diagonal: 160 degree (while other normal cameras are typically 72 degree) -->
-          <!-- <horizontal_fov>1.085595</horizontal_fov> -->
-          <horizontal_fov>1.2</horizontal_fov>
-          <image>
-              <width>420</width>
-              <height>240</height>
-              <format>R8G8B8</format>
-          </image>
-		 <!-- Distance in meters from the pose of the sensor to the closest point on the near clip plane -->
-          <clip>
-              <near>0.03</near>
-              <far>1.5</far>
-          </clip>
+  <gazebo reference="camera">
+    <sensor type="camera" name="cam">
+      <update_rate>10</update_rate>
+      <camera name="head">
+        <!-- The horizontal field of view of the camera in radians -->
+        <!-- Pi Fisheye Diagonal: 160 degree (while other normal cameras are typically 72 degree) -->
+        <!-- <horizontal_fov>1.085595</horizontal_fov> -->
+        <horizontal_fov>1.2</horizontal_fov>
+        <image>
+          <width>420</width>
+          <height>240</height>
+          <format>R8G8B8</format>
+        </image>
+        <!-- Distance in meters from the pose of the sensor to the closest point on the near clip plane -->
+        <clip>
+          <near>0.02</near>
+          <far>300</far>
+        </clip>
       </camera>
       <plugin name="camera_controller" filename="libgazebo_ros_camera.so">
         <alwaysOn>true</alwaysOn>
-        <updateRate>1.0</updateRate>
+        <updateRate>10.0</updateRate>
         <cameraName>camera</cameraName>
-        <frameName>camera_optical</frameName>
+        <frameName>camera</frameName>
         <imageTopicName>image</imageTopicName>
-        <cameraInfoTopicName>camerainfo</cameraInfoTopicName>
+        <cameraInfoTopicName>camera_info</cameraInfoTopicName>
         <hackBaseline>0.07</hackBaseline>
         <distortionK1>0.0</distortionK1>
@@ -232,5 +228,5 @@
   </joint>
   <joint name="camera_joint" type="fixed">
-	<origin xyz="-0.07 0 0.65" rpy="0 0.9 0"/>
+	  <origin xyz="-0.07 0 0.65" rpy="0 0.9 0"/>
     <parent link="base_link"/>
     <child link="camera"/>
@@ -251,15 +247,3 @@
     </collision>
   </link>
-  <joint name="camera_rgb_joint" type="fixed">
-    <origin xyz="0 0 0" rpy="0 0 0"/>
-    <parent link="camera"/>
-    <child link="camera_rgb_frame"/>
-  </joint>
-  <link name="camera_rgb_frame"/>
-  <joint name="camera_optical" type="fixed">
-    <origin xyz="0 0 0" rpy="-1.57 0 -1.57"/>
-    <parent link="camera_rgb_frame"/>
-    <child link="camera_optical"/>
-  </joint>
-  <link name="camera_optical"/>
 </robot>

Commit message: migrating camera plugin to ROS2

File: dev_ws/src/field_robot/robot_description/tb3/turtlebot3_burger_for_pumpkin.urdf.xacro (robot description, xacro)
@@ -32,5 +32,129 @@
     <color rgba="1.0 1.0 1.0 1.0"/>
   </material>
-  <gazebo reference="base_link">
+  <link name="base_footprint"/>
+  <link name="base_link">
+    <visual>
+      <origin xyz="-0.032 0 0.0" rpy="0 0 0"/>
+      <geometry>
+        <mesh filename="model://tb3/bases/burger_base.stl" scale="0.001 0.001 0.001"/>
+      </geometry>
+      <material name="light_black"/>
+    </visual>
+    <collision>
+      <origin xyz="-0.032 0 0.070" rpy="0 0 0"/>
+      <geometry>
+        <box size="0.140 0.140 0.143"/>
+      </geometry>
+    </collision>
+    <inertial>
+      <origin xyz="0 0 0" rpy="0 0 0"/>
+      <mass value="8.2573504e-01"/>
+      <inertia ixx="2.2124416e-03" ixy="-1.2294101e-05" ixz="3.4938785e-05"
+               iyy="2.1193702e-03" iyz="-5.0120904e-06"
+               izz="2.0064271e-03" />
+    </inertial>
+  </link>
+  <joint name="base_joint" type="fixed">
+    <parent link="base_footprint"/>
+    <child link="base_link"/>
+    <origin xyz="0.0 0.0 0.010" rpy="0 0 0"/>
+  </joint>
+  <!--<link name="wheel_l">
+    <visual>
+      <origin xyz="0 0 0" rpy="1.57 0 0"/>
+      <geometry>
+        <mesh filename="model://tb3/wheels/left_tire.stl" scale="0.001 0.001 0.001"/>
+      </geometry>
+      <material name="dark"/>
+    </visual>
+    <collision>
+      <origin xyz="0 0 0" rpy="0 0 0"/>
+      <geometry>
+        <cylinder length="0.018" radius="0.033"/>
+      </geometry>
+    </collision>
+    <inertial>
+      <origin xyz="0 0 0" />
+      <mass value="2.8498940e-02" />
+      <inertia ixx="1.1175580e-05" ixy="-4.2369783e-11" ixz="-5.9381719e-09"
+               iyy="1.1192413e-05" iyz="-1.4400107e-11"
+               izz="2.0712558e-05" />
+      </inertial>
+  </link>
+  <joint name="wheel_l_joint" type="continuous">
+    <parent link="base_link"/>
+    <child link="wheel_l"/>
+    <origin xyz="0.0 0.08 0.023" rpy="-1.57 0 0"/>
+    <axis xyz="0 0 1"/>
+  </joint>
+  <link name="wheel_r">
+    <visual>
+      <origin xyz="0 0 0" rpy="1.57 0 0"/>
+      <geometry>
+        <mesh filename="model://tb3/wheels/right_tire.stl" scale="0.001 0.001 0.001"/>
+      </geometry>
+      <material name="dark"/>
+    </visual>
+    <collision>
+      <origin xyz="0 0 0" rpy="0 0 0"/>
+      <geometry>
+        <cylinder length="0.018" radius="0.033"/>
+      </geometry>
+    </collision>
+    <inertial>
+      <origin xyz="0 0 0" />
+      <mass value="2.8498940e-02" />
+      <inertia ixx="1.1175580e-05" ixy="-4.2369783e-11" ixz="-5.9381719e-09"
+               iyy="1.1192413e-05" iyz="-1.4400107e-11"
+               izz="2.0712558e-05" />
+      </inertial>
+  </link>
+  <joint name="wheel_r_joint" type="continuous">
+    <parent link="base_link"/>
+    <child link="wheel_r"/>
+    <origin xyz="0.0 -0.080 0.023" rpy="-1.57 0 0"/>
+    <axis xyz="0 0 1"/>
+  </joint>
+  <link name="caster_back_link">
+    <collision>
+      <origin xyz="0 0.001 0" rpy="0 0 0"/>
+      <geometry>
+        <box size="0.030 0.009 0.020"/>
+      </geometry>
+    </collision>
+    <inertial>
+      <origin xyz="0 0 0" />
+      <mass value="0.005" />
+      <inertia ixx="0.001" ixy="0.0" ixz="0.0"
+               iyy="0.001" iyz="0.0"
+               izz="0.001" />
+    </inertial>
+  </link>
+  <joint name="caster_back_joint" type="fixed">
+    <parent link="base_link"/>
+    <child link="caster_back_link"/>
+    <origin xyz="-0.081 0 -0.004" rpy="-1.57 0 0"/>
+  </joint>-->
+  <link name="camera_link">
+    <visual>
+      <origin xyz="0 0 0" rpy="0 0 0"/>
+      <geometry>
+        <box size="0.015 0.030 0.027"/>
+      </geometry>
+      <material name="dark"/>
+    </visual>
+    <collision>
+      <origin xyz="0 0 0" rpy="0 0 0"/>
+      <geometry>
+        <box size="0.015 0.030 0.027"/>
+      </geometry>
+    </collision>
+  </link>
+  <joint name="camera_joint" type="fixed">
+	  <origin xyz="-0.07 0 0.65" rpy="0 0.9 0"/>
+    <parent link="base_link"/>
+    <child link="camera_link"/>
+  </joint>
+  <!-- <gazebo reference="base_link">
     <material>Gazebo/DarkGrey</material>
   </gazebo>
@@ -66,7 +190,5 @@
   <gazebo>
     <plugin name="turtlebot3_burger_controller" filename="libgazebo_ros_diff_drive.so">
-      <commandTopic>cmd_vel</commandTopic>
-      <odometryTopic>odom</odometryTopic>
-      <odometryFrame>odom</odometryFrame>
+      <odometry_frame>odom</odometry_frame>
       <odometrySource>odom</odometrySource>
       <publishOdomTF>true</publishOdomTF>
@@ -76,18 +198,22 @@
       <publishWheelJointState>false</publishWheelJointState>
       <legacyMode>false</legacyMode>
-      <updateRate>30</updateRate>
+      <update_rate>30</update_rate>
       <left_joint>wheel_l_joint</left_joint>
       <right_joint>wheel_r_joint</right_joint>
       <wheel_separation>0.160</wheel_separation>
       <wheel_diameter>0.066</wheel_diameter>
-      <wheelAcceleration>1</wheelAcceleration>
-      <wheelTorque>10</wheelTorque>
+      <max_wheel_acceleration>1</max_wheel_acceleration>
+      <max_wheel_torque>10</max_wheel_torque>
       <rosDebugLevel>na</rosDebugLevel>
+      <ros>
+        <argument>cmd_vel:=custom_cmd_vel</argument>
+        <argument>odom:=custom_odom</argument>
+      </ros>
     </plugin>
-  </gazebo>
+  </gazebo> -->
   <!--link : https://www.raspberrypi.org/documentation/hardware/camera/-->
-  <gazebo reference="camera">
-    <sensor type="camera" name="cam">
-      <update_rate>10</update_rate>
+  <gazebo reference="camera_link">
+    <sensor type="camera" name="camera1">
+      <update_rate>1</update_rate>
       <camera name="head">
         <!-- The horizontal field of view of the camera in radians -->
@@ -105,145 +231,24 @@
           <far>300</far>
         </clip>
+        <distortion>
+          <k1>0.0</k1>
+          <k2>0.0</k2>
+          <k3>0.0</k3>
+          <p1>0.0</p1>
+          <p2>0.0</p2>
+        </distortion>
       </camera>
       <plugin name="camera_controller" filename="libgazebo_ros_camera.so">
-        <alwaysOn>true</alwaysOn>
-        <updateRate>10.0</updateRate>
-        <cameraName>camera</cameraName>
-        <frameName>camera</frameName>
-        <imageTopicName>image</imageTopicName>
-        <cameraInfoTopicName>camera_info</cameraInfoTopicName>
-        <hackBaseline>0.07</hackBaseline>
-        <distortionK1>0.0</distortionK1>
-        <distortionK2>0.0</distortionK2>
-        <distortionK3>0.0</distortionK3>
-        <distortionT1>0.0</distortionT1>
-        <distortionT2>0.0</distortionT2>
+        <ros>
+          <namespace>custom_ns</namespace>
+          <argument>image_raw:=custom</argument>
+          <argument>camera_info:=custom_info</argument>
+        </ros>
+        <camera_name>camera1</camera_name>
+        <frame_name>camera_link</frame_name>
+        <hack_baseline>0.07</hack_baseline>
       </plugin>
     </sensor>
   </gazebo>
   <!-- ENDE ENDE ENDE ENDE-->
-  <link name="base_footprint"/>
-  <joint name="base_joint" type="fixed">
-    <parent link="base_footprint"/>
-    <child link="base_link"/>
-    <origin xyz="0.0 0.0 0.010" rpy="0 0 0"/>
-  </joint>
-  <link name="base_link">
-    <visual>
-      <origin xyz="-0.032 0 0.0" rpy="0 0 0"/>
-      <geometry>
-        <mesh filename="model://tb3/bases/burger_base.stl" scale="0.001 0.001 0.001"/>
-      </geometry>
-      <material name="light_black"/>
-    </visual>
-    <collision>
-      <origin xyz="-0.032 0 0.070" rpy="0 0 0"/>
-      <geometry>
-        <box size="0.140 0.140 0.143"/>
-      </geometry>
-    </collision>
-    <inertial>
-      <origin xyz="0 0 0" rpy="0 0 0"/>
-      <mass value="8.2573504e-01"/>
-      <inertia ixx="2.2124416e-03" ixy="-1.2294101e-05" ixz="3.4938785e-05"
-               iyy="2.1193702e-03" iyz="-5.0120904e-06"
-               izz="2.0064271e-03" />
-    </inertial>
-  </link>
-  <link name="wheel_l">
-    <visual>
-      <origin xyz="0 0 0" rpy="1.57 0 0"/>
-      <geometry>
-        <mesh filename="model://tb3/wheels/left_tire.stl" scale="0.001 0.001 0.001"/>
-      </geometry>
-      <material name="dark"/>
-    </visual>
-    <collision>
-      <origin xyz="0 0 0" rpy="0 0 0"/>
-      <geometry>
-        <cylinder length="0.018" radius="0.033"/>
-      </geometry>
-    </collision>
-    <inertial>
-      <origin xyz="0 0 0" />
-      <mass value="2.8498940e-02" />
-      <inertia ixx="1.1175580e-05" ixy="-4.2369783e-11" ixz="-5.9381719e-09"
-               iyy="1.1192413e-05" iyz="-1.4400107e-11"
-               izz="2.0712558e-05" />
-      </inertial>
-  </link>
-  <joint name="wheel_l_joint" type="continuous">
-    <parent link="base_link"/>
-    <child link="wheel_l"/>
-    <origin xyz="0.0 0.08 0.023" rpy="-1.57 0 0"/>
-    <axis xyz="0 0 1"/>
-  </joint>
-  <link name="wheel_r">
-    <visual>
-      <origin xyz="0 0 0" rpy="1.57 0 0"/>
-      <geometry>
-        <mesh filename="model://tb3/wheels/right_tire.stl" scale="0.001 0.001 0.001"/>
-      </geometry>
-      <material name="dark"/>
-    </visual>
-    <collision>
-      <origin xyz="0 0 0" rpy="0 0 0"/>
-      <geometry>
-        <cylinder length="0.018" radius="0.033"/>
-      </geometry>
-    </collision>
-    <inertial>
-      <origin xyz="0 0 0" />
-      <mass value="2.8498940e-02" />
-      <inertia ixx="1.1175580e-05" ixy="-4.2369783e-11" ixz="-5.9381719e-09"
-               iyy="1.1192413e-05" iyz="-1.4400107e-11"
-               izz="2.0712558e-05" />
-      </inertial>
-  </link>
-  <joint name="wheel_r_joint" type="continuous">
-    <parent link="base_link"/>
-    <child link="wheel_r"/>
-    <origin xyz="0.0 -0.080 0.023" rpy="-1.57 0 0"/>
-    <axis xyz="0 0 1"/>
-  </joint>
-  <link name="caster_back_link">
-    <collision>
-      <origin xyz="0 0.001 0" rpy="0 0 0"/>
-      <geometry>
-        <box size="0.030 0.009 0.020"/>
-      </geometry>
-    </collision>
-    <inertial>
-      <origin xyz="0 0 0" />
-      <mass value="0.005" />
-      <inertia ixx="0.001" ixy="0.0" ixz="0.0"
-               iyy="0.001" iyz="0.0"
-               izz="0.001" />
-    </inertial>
-  </link>
-  <joint name="caster_back_joint" type="fixed">
-    <parent link="base_link"/>
-    <child link="caster_back_link"/>
-    <origin xyz="-0.081 0 -0.004" rpy="-1.57 0 0"/>
-  </joint>
-  <joint name="camera_joint" type="fixed">
-	  <origin xyz="-0.07 0 0.65" rpy="0 0.9 0"/>
-    <parent link="base_link"/>
-    <child link="camera"/>
-  </joint>
-  <link name="camera">
-    <visual>
-      <origin xyz="0 0 0" rpy="0 0 0"/>
-      <geometry>
-        <box size="0.015 0.030 0.027"/>
-      </geometry>
-      <material name="dark"/>
-    </visual>
-    <collision>
-      <origin xyz="0 0 0" rpy="0 0 0"/>
-      <geometry>
-        <box size="0.015 0.030 0.027"/>
-      </geometry>
-    </collision>
-  </link>
 </robot>

Commit message: updating the robot description, trying to get the camera working

File: dev_ws/src/field_robot/robot_description/tb3/turtlebot3_burger_for_pumpkin.urdf.xacro (robot description, xacro)
@@ -60,5 +60,5 @@
     <origin xyz="0.0 0.0 0.010" rpy="0 0 0"/>
   </joint>
-  <!--<link name="wheel_l">
+  <link name="wheel_l">
     <visual>
       <origin xyz="0 0 0" rpy="1.57 0 0"/>
@@ -135,5 +135,5 @@
     <child link="caster_back_link"/>
     <origin xyz="-0.081 0 -0.004" rpy="-1.57 0 0"/>
-  </joint>-->
+  </joint>
   <link name="camera_link">
     <visual>
@@ -156,5 +156,5 @@
     <child link="camera_link"/>
   </joint>
-  <!-- <gazebo reference="base_link">
+  <gazebo reference="base_link">
     <material>Gazebo/DarkGrey</material>
   </gazebo>
@@ -189,4 +189,8 @@
   </gazebo>
   <gazebo>
+    <plugin name="joint_states" filename="libgazebo_ros_joint_state_publisher.so">
+      <joint_name>wheel_l_joint</joint_name>
+      <joint_name>wheel_r_joint</joint_name>
+    </plugin>
     <plugin name="turtlebot3_burger_controller" filename="libgazebo_ros_diff_drive.so">
       <odometry_frame>odom</odometry_frame>
@@ -196,5 +200,4 @@
       <publishWheelTF>false</publishWheelTF>
       <publishTf>true</publishTf>
-      <publishWheelJointState>false</publishWheelJointState>
       <legacyMode>false</legacyMode>
       <update_rate>30</update_rate>
@@ -206,13 +209,14 @@
       <max_wheel_torque>10</max_wheel_torque>
       <rosDebugLevel>na</rosDebugLevel>
-      <ros>
+      <!--<ros>
         <argument>cmd_vel:=custom_cmd_vel</argument>
         <argument>odom:=custom_odom</argument>
-      </ros>
+      </ros>-->
     </plugin>
-  </gazebo> -->
+  </gazebo>
   <!--link : https://www.raspberrypi.org/documentation/hardware/camera/-->
   <gazebo reference="camera_link">
     <sensor type="camera" name="camera1">
+      <always_on>0</always_on>
       <update_rate>1</update_rate>
       <camera name="head">
@@ -240,10 +244,10 @@
       </camera>
       <plugin name="camera_controller" filename="libgazebo_ros_camera.so">
-        <ros>
+        <!--<ros>
           <namespace>custom_ns</namespace>
           <argument>image_raw:=custom</argument>
           <argument>camera_info:=custom_info</argument>
-        </ros>
-        <camera_name>camera1</camera_name>
+        </ros> -->
+        <camera_name>camera2</camera_name>
         <frame_name>camera_link</frame_name>
         <hack_baseline>0.07</hack_baseline>

Commit message: added the scanner to the simulation and did changed necessary for the setup to work, including adjusting the crop size to be recognized

File: dev_ws/src/field_robot/robot_description/tb3/turtlebot3_burger_for_pumpkin.urdf.xacro (robot description, xacro)
@@ -58,4 +58,10 @@
     <child link="base_link"/>
     <origin xyz="0.0 0.0 0.010" rpy="0 0 0"/>
+  </joint>
+  <link name="scanner_link"/>
+  <joint name="scanner_joint" type="fixed">
+    <parent link="base_link"/>
+    <child link="scanner_link"/>
+    <origin xyz="0.0 0.0 0.25" rpy="0 0 0"/>
   </joint>
   <link name="wheel_l">
@@ -255,4 +261,40 @@
     </sensor>
   </gazebo>
+  <gazebo reference="scanner_link">
+    <sensor name="laser_scanner" type="ray">
+      <always_on>true</always_on>
+      <visualize>true</visualize>
+      <pose>0 0 0 0 0 0</pose>
+      <update_rate>5</update_rate>
+      <ray>
+        <scan>
+          <horizontal>
+            <samples>360</samples>
+            <resolution>1.000000</resolution>
+            <min_angle>0.000000</min_angle>
+            <max_angle>6.280000</max_angle>
+          </horizontal>
+        </scan>
+        <range>
+          <min>0.120000</min>
+          <max>3.5</max>
+          <resolution>0.015000</resolution>
+        </range>
+        <noise>
+          <type>gaussian</type>
+          <mean>0.0</mean>
+          <stddev>0.01</stddev>
+        </noise>
+      </ray>
+      <plugin name="tb3_laserscanner" filename="libgazebo_ros_ray_sensor.so">
+        <ros>
+          <namespace>field_robot</namespace>
+          <remapping>~/out:=scan</remapping>
+        </ros>
+        <output_type>sensor_msgs/LaserScan</output_type>
+        <frame_name>scanner_link</frame_name>
+      </plugin>
+    </sensor>
+  </gazebo>
   <!--<gazebo>
     <plugin name="gaezbo_ros_p3d" filename="libgazebo_ros_p3d.so">
