Commit message: updating the robot model

File: dev_ws/src/virtual_maize_field/models/robot/robot.urdf (robot description, URDF)
Before this commit: robot robot, 10 links, 9 joints
Links:
- added link camera_back_virtual_link
- added link camera_front_virtual_link
- added link camera_left_virtual_link
- added link camera_right_virtual_link
Joints:
- added joint camera_back_virtual_joint: type fixed, parent camera_back_link, child camera_back_virtual_link, origin xyz=0 0 0 rpy=1.57079632679 -1.57079632679 0
- added joint camera_front_virtual_joint: type fixed, parent camera_front_link, child camera_front_virtual_link, origin xyz=0 0 0 rpy=1.57079632679 -1.57079632679 0
- added joint camera_left_virtual_joint: type fixed, parent camera_left_link, child camera_left_virtual_link, origin xyz=0 0 0 rpy=1.57079632679 -1.57079632679 0
- added joint camera_right_virtual_joint: type fixed, parent camera_right_link, child camera_right_virtual_link, origin xyz=0 0 0 rpy=1.57079632679 -1.57079632679 0
- joint camera_back_joint: origin xyz=-0.15 0.0 0.1 rpy=0 0 3.14159265 -> xyz=-0.15 0.0 0.1 rpy=-1.57079632679 0 1.57079632679
- joint camera_front_joint: origin xyz=0.15 0.0 0.1 rpy=0 0 0 -> xyz=0.15 0.0 0.1 rpy=-1.57079632679 0 -1.57079632679
- joint camera_left_joint: origin xyz=0.0 0.15 0.1 rpy=0 0 1.5708 -> xyz=0.0 0.15 0.1 rpy=-1.57079632679 0 0
- joint camera_right_joint: origin xyz=0.0 -0.15 0.1 rpy=0 0 -1.5708 -> xyz=0.0 -0.15 0.1 rpy=-1.57079632679 0 3.1415926536
- joint caster_back_joint: origin xyz=-0.4 0.0 -0.12 rpy=-1.57 0 0 -> xyz=-0.4 0.0 -0.12 rpy=-1.57079632679 0 0
- joint wheel_l_joint: origin xyz=0.0 0.125 0.0 rpy=-1.57 0 0 -> xyz=0.0 0.125 0.0 rpy=-1.57079632679 0 0
- joint wheel_r_joint: origin xyz=0.0 -0.125 0.0 rpy=-1.57 0 0 -> xyz=0.0 -0.125 0.0 rpy=-1.57079632679 0 0
