Commit message: updating the robot model according to the physicial robot & starting configuration of the simulation

File: dev_ws/src/field_robot/models/robot/robot.urdf (robot description, URDF)
Before this commit: robot robot, 7 links, 6 joints
Links:
- removed link camera_link
- removed link scanner_link
- link base_link: mass 8.2573504e-01 -> 1; geometry collision box size=0.2 0.2 0.2; visual box size=0.2 0.2 0.2
- link caster_back_link: mass 0.005 -> 6; geometry collision cylinder length=0.045 radius=0.02; visual cylinder length=0.045 radius=0.02
- link wheel_l: mass 2.8498940e-02 -> 4; geometry collision cylinder length=0.045 radius=0.2; visual cylinder length=0.045 radius=0.2
- link wheel_r: mass 2.8498940e-02 -> 4; geometry collision cylinder length=0.045 radius=0.2; visual cylinder length=0.045 radius=0.2
Joints:
- removed joint camera_joint
- removed joint scanner_joint
- joint base_joint: origin xyz=0.0 0.0 0.010 rpy=0 0 0 -> xyz=0.0 0.0 0.2 rpy=0 0 0
- joint caster_back_joint: origin xyz=-0.081 0 -0.004 rpy=-1.57 0 0 -> xyz=-0.4 0.0 -0.19 rpy=-1.57 0 0
- joint wheel_l_joint: origin xyz=0.0 0.08 0.023 rpy=-1.57 0 0 -> xyz=0.0 0.125 0.0 rpy=-1.57 0 0
- joint wheel_r_joint: origin xyz=0.0 -0.080 0.023 rpy=-1.57 0 0 -> xyz=0.0 -0.125 0.0 rpy=-1.57 0 0

Commit message: adding a build script and updating the robot model with inertia details

File: dev_ws/src/field_robot/models/robot/robot.urdf (robot description, URDF)
Before this commit: robot robot, 5 links, 4 joints
Links:
- link caster_back_link: mass 6 -> 4
Joints:
- joint wheel_r_joint: origin xyz=0.0 -0.125 0.0 rpy=-1.57 0 0 -> xyz=0.0 -0.125 0.0 rpy=1.57 0 0

Commit message: updating roobt model

File: dev_ws/src/field_robot/models/robot/robot.urdf (robot description, URDF)
Before this commit: robot robot, 5 links, 4 joints
Joints:
- joint wheel_r_joint: origin xyz=0.0 -0.125 0.0 rpy=1.57 0 0 -> xyz=0.0 -0.125 0.0 rpy=-1.57 0 0

Commit message: updating robot model

File: dev_ws/src/field_robot/models/robot/robot.urdf (robot description, URDF)
Before this commit: robot robot, 5 links, 4 joints
Links:
- link caster_back_link: geometry collision sphere radius=0.08; visual sphere radius=0.08
Joints:
- joint caster_back_joint: origin xyz=-0.4 0.0 -0.19 rpy=-1.57 0 0 -> xyz=-0.4 0.0 -0.12 rpy=-1.57 0 0

Commit message: updatin simulation parameters and adding four cameras

File: dev_ws/src/field_robot/models/robot/robot.urdf (robot description, URDF)
Before this commit: robot robot, 5 links, 4 joints
Links:
- added link camera_back_link, mass 0; collision box size=0.005 0.1 0.02; visual box size=0.005 0.1 0.02
- added link camera_front_link, mass 0; collision box size=0.005 0.1 0.02; visual box size=0.005 0.1 0.02
- added link camera_left_link, mass 0; collision box size=0.005 0.1 0.02; visual box size=0.005 0.1 0.02
- added link camera_right_link, mass 0; collision box size=0.005 0.1 0.02; visual box size=0.005 0.1 0.02
Joints:
- added joint camera_back_joint: type fixed, parent base_link, child camera_back_link, origin xyz=-0.15 0.0 0.1 rpy=0 0 3.14159265
- added joint camera_front_joint: type fixed, parent base_link, child camera_front_link, origin xyz=0.15 0.0 0.1 rpy=0 0 0
- added joint camera_left_joint: type fixed, parent base_link, child camera_left_link, origin xyz=0.0 0.15 0.1 rpy=0 0 1.5708
- added joint camera_right_joint: type fixed, parent base_link, child camera_right_link, origin xyz=0.0 -0.15 0.1 rpy=0 0 -1.5708

Commit message: adding the imu and updating the camera integration

File: dev_ws/src/field_robot/models/robot/robot.urdf (robot description, URDF)
Before this commit: robot robot, 9 links, 8 joints
Links:
- added link imu_link, mass 0; collision box size=0.05 0.05 0.05; visual box size=0.05 0.05 0.05
Joints:
- added joint imu_join: type fixed, parent base_link, child imu_link, origin xyz=0 0 0 rpy=0 0 0

Commit message: disabling all but the front camera

File: dev_ws/src/field_robot/models/robot/robot.urdf (robot description, URDF)
Before this commit: robot robot, 10 links, 9 joints
Links:
- removed link camera_left_link
- removed link camera_right_link
Joints:
- removed joint camera_left_joint
- removed joint camera_right_joint

Commit message: rotating camera

File: dev_ws/src/field_robot/models/robot/robot.urdf (robot description, URDF)
Before this commit: robot robot, 8 links, 7 joints
Joints:
- joint camera_front_joint: origin xyz=0.15 0.0 0.1 rpy=0 0 0 -> xyz=0.15 0.0 0.1 rpy=-1.5708 0 0

Commit message: updating camera frames and camera sensor positioning
Now, the frame uses the correct orientation as used in the inverted image projection and as defined by ROS. Accordingly, also reference frame for the gazebo camera sensor had to be updated to still keep the same image while modifying the frame rotation.

File: dev_ws/src/field_robot/models/robot/robot.urdf (robot description, URDF)
Before this commit: robot robot, 8 links, 7 joints
Links:
- added link camera_back_virtual_link
- added link camera_front_virtual_link
Joints:
- added joint camera_back_virtual_joint: type fixed, parent camera_back_link, child camera_back_virtual_link, origin xyz=0 0 0 rpy=0 -1.5708 1.5708
- added joint camera_front_virtual_joint: type fixed, parent camera_front_link, child camera_front_virtual_link, origin xyz=0 0 0 rpy=0 -1.5708 1.5708
- joint camera_back_joint: origin xyz=-0.15 0.0 0.1 rpy=0 0 3.14159265 -> xyz=-0.15 0.0 0.1 rpy=-1.5708 0 -1.5708
- joint camera_front_joint: origin xyz=0.15 0.0 0.1 rpy=-1.5708 0 0 -> xyz=0.15 0.0 0.1 rpy=-1.5708 0 -1.5708

Commit message: updating pi/2 accuracy

File: dev_ws/src/field_robot/models/robot/robot.urdf (robot description, URDF)
Before this commit: robot robot, 10 links, 9 joints
Joints:
- joint camera_back_joint: origin xyz=-0.15 0.0 0.1 rpy=-1.5708 0 -1.5708 -> xyz=-0.15 0.0 0.1 rpy=-1.57079632679 0 -1.57079632679
- joint camera_back_virtual_joint: origin xyz=0 0 0 rpy=0 -1.5708 1.5708 -> xyz=0 0 0 rpy=0 -1.57079632679 1.57079632679
- joint camera_front_joint: origin xyz=0.15 0.0 0.1 rpy=-1.5708 0 -1.5708 -> xyz=0.15 0.0 0.1 rpy=-1.57079632679 0 -1.57079632679
- joint camera_front_virtual_joint: origin xyz=0 0 0 rpy=0 -1.5708 1.5708 -> xyz=0 0 0 rpy=0 -1.57079632679 1.57079632679
- joint caster_back_joint: origin xyz=-0.4 0.0 -0.12 rpy=-1.57 0 0 -> xyz=-0.4 0.0 -0.12 rpy=-1.57079632679 0 0
- joint wheel_l_joint: origin xyz=0.0 0.125 0.0 rpy=-1.57 0 0 -> xyz=0.0 0.125 0.0 rpy=-1.57079632679 0 0
- joint wheel_r_joint: origin xyz=0.0 -0.125 0.0 rpy=-1.57 0 0 -> xyz=0.0 -0.125 0.0 rpy=-1.57079632679 0 0

Commit message: updating camera positioning
Earlier changes accidentally oriented all cameras to the same direction leading to bugged images.

File: dev_ws/src/field_robot/models/robot/robot.urdf (robot description, URDF)
Before this commit: robot robot, 10 links, 9 joints
Links:
- added link camera_left_link, mass 0; collision box size=0.005 0.1 0.02; visual box size=0.005 0.1 0.02
- added link camera_left_virtual_link
- added link camera_right_link, mass 0; collision box size=0.005 0.1 0.02; visual box size=0.005 0.1 0.02
- added link camera_right_virtual_link
Joints:
- added joint camera_left_joint: type fixed, parent base_link, child camera_left_link, origin xyz=0.0 0.15 0.1 rpy=0 0 1.57079632679
- added joint camera_left_virtual_joint: type fixed, parent camera_left_link, child camera_left_virtual_link, origin xyz=0 0 0 rpy=0 -1.57079632679 1.57079632679
- added joint camera_right_joint: type fixed, parent base_link, child camera_right_link, origin xyz=0.0 -0.15 0.1 rpy=0 0 -1.57079632679
- added joint camera_right_virtual_joint: type fixed, parent camera_right_link, child camera_right_virtual_link, origin xyz=0 0 0 rpy=0 -1.57079632679 1.57079632679
- joint camera_back_joint: origin xyz=-0.15 0.0 0.1 rpy=-1.57079632679 0 -1.57079632679 -> xyz=-0.15 0.0 0.1 rpy=0 0 3.1415926536

Commit message: rotating faulty camera

File: dev_ws/src/field_robot/models/robot/robot.urdf (robot description, URDF)
Before this commit: robot robot, 14 links, 13 joints
Joints:
- joint camera_front_joint: origin xyz=0.15 0.0 0.1 rpy=-1.57079632679 0 -1.57079632679 -> xyz=0.15 0.0 0.1 rpy=0 0 0

Commit message: updating camera rotation

File: dev_ws/src/field_robot/models/robot/robot.urdf (robot description, URDF)
Before this commit: robot robot, 14 links, 13 joints
Joints:
- joint camera_back_joint: origin xyz=-0.15 0.0 0.1 rpy=0 0 3.1415926536 -> xyz=-0.15 0.0 0.1 rpy=-1.57079632679 0 1.57079632679
- joint camera_back_virtual_joint: origin xyz=0 0 0 rpy=0 -1.57079632679 1.57079632679 -> xyz=0 0 0 rpy=1.57079632679 -1.57079632679 0
- joint camera_front_joint: origin xyz=0.15 0.0 0.1 rpy=0 0 0 -> xyz=0.15 0.0 0.1 rpy=-1.57079632679 0 -1.57079632679
- joint camera_front_virtual_joint: origin xyz=0 0 0 rpy=0 -1.57079632679 1.57079632679 -> xyz=0 0 0 rpy=1.57079632679 -1.57079632679 0
- joint camera_left_joint: origin xyz=0.0 0.15 0.1 rpy=0 0 1.57079632679 -> xyz=0.0 0.15 0.1 rpy=-1.57079632679 0 0
- joint camera_left_virtual_joint: origin xyz=0 0 0 rpy=0 -1.57079632679 1.57079632679 -> xyz=0 0 0 rpy=1.57079632679 -1.57079632679 0
- joint camera_right_joint: origin xyz=0.0 -0.15 0.1 rpy=0 0 -1.57079632679 -> xyz=0.0 -0.15 0.1 rpy=-1.57079632679 0 3.1415926536
- joint camera_right_virtual_joint: origin xyz=0 0 0 rpy=0 -1.57079632679 1.57079632679 -> xyz=0 0 0 rpy=1.57079632679 -1.57079632679 0

Commit message: updated robot model

File: dev_ws/src/field_robot/models/robot/robot.urdf (robot description, URDF)
Before this commit: robot robot, 15 links, 14 joints
Links:
- removed link caster_back_link
- removed link lidar_link
- removed link wheel_l
- removed link wheel_r
- added link wheel_lb, mass 4; collision cylinder length=0.06 radius=0.123345; visual cylinder length=0.06 radius=0.123345
- added link wheel_lf, mass 4; collision cylinder length=0.055 radius=0.123345; visual cylinder length=0.055 radius=0.123345
- added link wheel_rb, mass 4; collision cylinder length=0.06 radius=0.123345; visual cylinder length=0.06 radius=0.123345
- added link wheel_rf, mass 4; collision cylinder length=0.055 radius=0.123345; visual cylinder length=0.055 radius=0.123345
- link base_link: mass 1 -> 10; geometry collision box size=0.4 0.21 0.05; visual box size=0.4 0.21 0.05
- link camera_back_link: mass 0 -> 1
- link camera_front_link: mass 0 -> 1
- link camera_left_link: mass 0 -> 1
- link camera_right_link: mass 0 -> 1
- link imu_link: mass 0 -> 1
Joints:
- removed joint caster_back_joint
- removed joint lidar_joint
- removed joint wheel_l_joint
- removed joint wheel_r_joint
- added joint wheel_lb_joint: type continuous, parent base_link, child wheel_lb, origin xyz=-0.1685 0.16 -0.035 rpy=-1.57079632679 0 0, axis 0 0 1
- added joint wheel_lf_joint: type continuous, parent base_link, child wheel_lf, origin xyz=0.1685 0.155 -0.035 rpy=-1.57079632679 0 0, axis 0 0 1
- added joint wheel_rb_joint: type continuous, parent base_link, child wheel_rb, origin xyz=-0.1685 -0.16 -0.035 rpy=-1.57079632679 0 0, axis 0 0 1
- added joint wheel_rf_joint: type continuous, parent base_link, child wheel_rf, origin xyz=0.1685 -0.155 -0.035 rpy=-1.57079632679 0 0, axis 0 0 1
- joint camera_back_joint: origin xyz=-0.15 0.0 0.1 rpy=-1.57079632679 0 1.57079632679 -> xyz=-0.25 0.0 0.1 rpy=-2.35619449 0 1.57079632679
- joint camera_front_joint: origin xyz=0.15 0.0 0.1 rpy=-1.57079632679 0 -1.57079632679 -> xyz=0.25 0.0 0.1 rpy=-2.35619449 0 -1.57079632679
- joint camera_left_joint: origin xyz=0.0 0.15 0.1 rpy=-1.57079632679 0 0 -> xyz=0.0 0.155 0.1 rpy=-2.35619449 0 0
- joint camera_right_joint: origin xyz=0.0 -0.15 0.1 rpy=-1.57079632679 0 3.1415926536 -> xyz=0.0 -0.155 0.1 rpy=-2.35619449 0 3.1415926536
- joint imu_join: origin xyz=0 0 0 rpy=0 0 0 -> xyz=0 0 1 rpy=0 0 0

Commit message: rew robot model

File: dev_ws/src/field_robot/models/robot/robot.urdf (robot description, URDF)
Before this commit: robot robot, 15 links, 14 joints
Links:
- link base_link: mass 10 -> 1
- link wheel_lb: mass 4 -> 3
- link wheel_lf: mass 4 -> 3
- link wheel_rb: mass 4 -> 3
- link wheel_rf: mass 4 -> 3
Joints:
- joint camera_back_joint: origin xyz=-0.25 0.0 0.1 rpy=-2.35619449 0 1.57079632679 -> xyz=-0.35 0.0 0.1 rpy=-2.35619449 0 1.57079632679
- joint camera_front_joint: origin xyz=0.25 0.0 0.1 rpy=-2.35619449 0 -1.57079632679 -> xyz=0.35 0.0 0.1 rpy=-2.35619449 0 -1.57079632679
- joint camera_left_joint: origin xyz=0.0 0.155 0.1 rpy=-2.35619449 0 0 -> xyz=0.0 0.25 0.1 rpy=-2.35619449 0 0
- joint camera_right_joint: origin xyz=0.0 -0.155 0.1 rpy=-2.35619449 0 3.1415926536 -> xyz=0.0 -0.25 0.1 rpy=-2.35619449 0 3.1415926536
- joint imu_join: origin xyz=0 0 1 rpy=0 0 0 -> xyz=0 0 0.1 rpy=0 0 0

Commit message: updating robot model for debugging

File: dev_ws/src/field_robot/models/robot/robot.urdf (robot description, URDF)
Before this commit: robot robot, 15 links, 14 joints
Links:
- link imu_link: mass 1 -> 0
